Commit message: Add files via upload

File: my_arm_description/urdf/robot_arm.xacro (robot description, xacro)
@@ -135,29 +135,29 @@
   <child link="Link1_1"/>
   <axis xyz="0 1 0"/>
-  <limit lower="-3.14" upper="3.14" effort="5.0" velocity="1.57" />
+  <limit lower="0.0" upper="3.14" effort="5.0" velocity="1.57" />
   <!-- <dynamics damping="0.5" friction="1.0"/> -->
 </joint>
 <joint name="joint_2" type="revolute">
-  <origin xyz="-0.02605 0.021381 0.0" rpy="0 0 0"/>
+  <origin xyz="-0.02605 0.021381 0.0" rpy="-1.57 0 0"/>
   <parent link="Link1_1"/>
   <child link="Link2_1"/>
-  <axis xyz="-1 0 0"/>
-  <limit lower="-1.57" upper="1.57" effort="5.0" velocity="1.57" />
+  <axis xyz="1 0 0"/>
+  <limit lower="0.0" upper="3.14" effort="5.0" velocity="1.57" />
   <!-- <dynamics damping="0.5" friction="1.0"/> -->
 </joint>
 <joint name="joint_3" type="revolute">
-  <origin xyz="0.0 0.1 0.0" rpy="0 0 0"/>
+  <origin xyz="0.0 0.1 0.0" rpy="3.14 0 0"/>
   <parent link="Link2_1"/>
   <child link="Link3_1"/>
-  <axis xyz="-1 0 0"/>
-  <limit lower="-2.2" upper="2.2" effort="5.0" velocity="1.57" />
+  <axis xyz="1 0 0"/>
+  <limit lower="0.52" upper="3.14" effort="5.0" velocity="1.57" />
   <!-- <dynamics damping="0.5" friction="1.0"/> -->
 </joint>
 <joint name="joint_4" type="revolute">
-  <origin xyz="-0.00155 0.091299 0.0035" rpy="0 0 0"/>
+  <origin xyz="-0.00155 0.091299 0.0035" rpy="-1.57 0 0"/>
   <parent link="Link3_1"/>
   <child link="Link4_1"/>
-  <axis xyz="-1 0 0"/>
-  <limit lower="-3.14" upper="1.2" effort="5.0" velocity="1.57" />
+  <axis xyz="1 0 0"/>
+  <limit lower="0.52" upper="3.14" effort="5.0" velocity="1.57" />
   <!-- <dynamics damping="0.5" friction="1.0"/> -->
 </joint>
@@ -169,9 +169,9 @@
 <!-- gripper -->
 <joint name="joint_5" type="revolute">
-  <origin xyz="0 0 0" rpy="1.57 0 -1.57"/>
+  <origin xyz="0 0 0" rpy="1.57 0.7 -1.57"/>
   <parent link="Link5_1"/>
   <child link="grip_base_link"/>
   <axis xyz="0 0 1"/>
-  <limit lower="-3.14" upper="3.14" effort="5.0" velocity="1.57" />
+  <limit lower="0.52" upper="2.26" effort="5.0" velocity="1.57" />
 </joint>
 <link
