Commit message: version 3

File: my_arm_description/urdf/arduino_arm.urdf (robot description, URDF)
Before this commit: robot robot_arm, 8 links, 7 joints
Links:
- added link hand_grip1, mass 0.000187045062582082; collision mesh filename=package://my_arm_description/meshes/gripper_meshes/hand_gri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; visual mesh filename=package://my_arm_description/meshes/gripper_meshes/hand_gri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
- added link hand_grip2, mass 0.000187045056346137; collision mesh filename=package://my_arm_description/meshes/gripper_meshes/hand_gri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; visual mesh filename=package://my_arm_description/meshes/gripper_meshes/hand_gri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
- added link hand_link1, mass 0.000142065726893586; collision mesh filename=package://my_arm_description/meshes/gripper_meshes/hand_lin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; visual mesh filename=package://my_arm_description/meshes/gripper_meshes/hand_lin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
- added link hand_link2, mass 0.000142065726893586; collision mesh filename=package://my_arm_description/meshes/gripper_meshes/hand_lin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; visual mesh filename=package://my_arm_description/meshes/gripper_meshes/hand_lin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
- added link mid_link1, mass 0.0000310995574287565; collision mesh filename=package://my_arm_description/meshes/gripper_meshes/mid_link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; visual mesh filename=package://my_arm_description/meshes/gripper_meshes/mid_link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
- added link mid_link2, mass 0.00003; collision mesh filename=package://my_arm_description/meshes/gripper_meshes/mid_link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; visual mesh filename=package://my_arm_description/meshes/gripper_meshes/mid_link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
- added link tool_link
Joints:
- added joint gripper_joint: type revolute, parent grip_base_link, child hand_link2, origin xyz=-0.013 0.00535 0.02625 rpy=1.5708 0 3.1416, axis 0 0 1, limit lower=-0.5 upper=0.5 effort=5.0 velocity=1.57
- added joint hand_grip_joint1: type revolute, parent hand_link1, child hand_grip1, origin xyz=-0.021122 0.019871 0 rpy=0 0 0, axis 0 0 1, limit lower=-0.5 upper=0.5 effort=5.0 velocity=1.57, mimic joint=gripper_joint multiplier=1
- added joint hand_grip_joint2: type revolute, parent hand_link2, child hand_grip2, origin xyz=0.021045 0.019953 0 rpy=0 0 0, axis 0 0 -1, limit lower=-0.4 upper=0.4 effort=5.0 velocity=1.57, mimic joint=gripper_joint multiplier=1
- added joint hand_joint1: type revolute, parent grip_base_link, child hand_link1, origin xyz=0.015 0.00535 0.02625 rpy=1.5708 0 3.1416, axis 0 0 1, limit lower=-0.5 upper=0.5 effort=5.0 velocity=1.57, mimic joint=gripper_joint multiplier=-1
- added joint mid_joint_1: type revolute, parent grip_base_link, child mid_link1, origin xyz=0.005 0.00535 0.04675 rpy=1.5708 0 3.1416, axis 0 0 -1, limit lower=-0.6 upper=0.6 effort=5.0 velocity=1.57, mimic joint=gripper_joint multiplier=1
- added joint mid_joint_2: type revolute, parent grip_base_link, child mid_link2, origin xyz=-0.005 0.00535 0.04675 rpy=1.5708 0 3.1416, axis 0 0 -1, limit lower=-0.6 upper=0.6 effort=5.0 velocity=1.57, mimic joint=gripper_joint multiplier=-1
- added joint tool_joint: type fixed, parent grip_base_link, child tool_link, origin xyz=0 0 0.1 rpy=0 0 0
- joint base_fixed_joint: origin xyz=0 0 0.2 rpy=0 0 0 -> xyz=0 0 0 rpy=0 0 1.57
- joint joint_1: origin xyz=0 0 0.06 rpy=1.57 0 0 -> xyz=0 0 0.06 rpy=1.57 0 3.14
- joint joint_2: origin xyz=-0.02605 0.021381 0.0 rpy=-1.57 0 0 -> xyz=-0.02605 0.021381 0.0 rpy=-1.7 0 0
- joint joint_3: origin xyz=0.0 0.1 0.0 rpy=3.14 0 0 -> xyz=0.0 0.1 0.0 rpy=3.8 0 0
- joint joint_5: limit lower=0.52 upper=2.26 effort=5.0 velocity=1.57 -> lower=0.0 upper=1.57 effort=5.0 velocity=1.57; origin xyz=0 0 0 rpy=1.57 0.7 -1.57 -> xyz=0 0 0 rpy=1.57 -1.57 -1.57

File: my_arm_description/urdf/robot_arm.xacro (robot description, xacro)
@@ -12,5 +12,5 @@
 <link name="base_link">
   <inertial>
-    <origin xyz="-0.0019226671084236508 0.03127199959893212 0.003074002176362074" rpy="0 0 0"/>
+    <origin xyz="-0.0019226671084236508 0.03127199959893212 0.003074002176362074" rpy="0 0 3.14"/>
     <mass value="0.1"/>
     <inertia ixx="0.0135" ixy="0.0" ixz="0.0" iyy="0.0135" iyz="0.0" izz="0.05"/>
@@ -136,5 +136,4 @@
   <axis xyz="0 1 0"/>
   <limit lower="0.0" upper="3.14" effort="5.0" velocity="1.57" />
-  <!-- <dynamics damping="0.5" friction="1.0"/> -->
 </joint>
 <joint name="joint_2" type="revolute">
@@ -144,5 +143,4 @@
   <axis xyz="1 0 0"/>
   <limit lower="0.0" upper="3.14" effort="5.0" velocity="1.57" />
-  <!-- <dynamics damping="0.5" friction="1.0"/> -->
 </joint>
 <joint name="joint_3" type="revolute">
@@ -152,5 +150,4 @@
   <axis xyz="1 0 0"/>
   <limit lower="0.52" upper="3.14" effort="5.0" velocity="1.57" />
-  <!-- <dynamics damping="0.5" friction="1.0"/> -->
 </joint>
 <joint name="joint_4" type="revolute">
@@ -160,5 +157,4 @@
   <axis xyz="1 0 0"/>
   <limit lower="0.52" upper="3.14" effort="5.0" velocity="1.57" />
-  <!-- <dynamics damping="0.5" friction="1.0"/> -->
 </joint>
 <joint name="joint_5_fixed" type="fixed">
